File: coolant-controller/coolant-controller.kicad_sch (KiCad schematic)
At the start: 21 parts, among them J1 Conn_02x10_Top_Bottom, U1 W25Q128JVS, U2 RP2040, Y1 Crystal_GND24

Commit message: Selected some devices
Parts:
- added U3, U4: BTS4310GXUMA1, Package_SO:SOIC-8_3.9x4.9mm_P1.27mm, symbol Power_Management:AUIPS1052G
Connections:
- new net: U4.7 (D1), U4.8 (D1)
- new net: U3.7 (D1), U3.8 (D1)
- new net: U3.5 (D2), U3.6 (D2)
- new net: U4.5 (D2), U4.6 (D2)
